Commit message: Fix launch and runtime bugs: xacro arg syntax, spawn -urdf flag, ca.fmax, Pose import

File: src/nmpc_swarm_demo/urdf/box_bot.urdf.xacro (robot description, xacro)
@@ -6,5 +6,5 @@
     gets a unique robot_name so its topics sit under /<robot_name>/...
   -->
-  <xacro:property name="robot_name" value="box_bot"/>
+  <xacro:arg name="robot_name" default="box_bot"/>
   <xacro:property name="chassis_length" value="0.30"/>
   <xacro:property name="chassis_width"  value="0.20"/>
@@ -21,5 +21,5 @@
     <color rgba="0.1 0.1 0.1 1.0"/>
   </material>
-  <link name="${robot_name}/base_link">
+  <link name="$(arg robot_name)/base_link">
     <visual>
       <geometry>
@@ -39,5 +39,5 @@
   </link>
   <!-- Left wheel -->
-  <link name="${robot_name}/left_wheel">
+  <link name="$(arg robot_name)/left_wheel">
     <visual>
       <geometry>
@@ -56,12 +56,12 @@
     </inertial>
   </link>
-  <joint name="${robot_name}/left_wheel_joint" type="continuous">
+  <joint name="$(arg robot_name)/left_wheel_joint" type="continuous">
     <origin xyz="0 ${track_width/2} ${-chassis_height/2 - wheel_width/2}" rpy="0 0 0"/>
-    <parent link="${robot_name}/base_link"/>
-    <child link="${robot_name}/left_wheel"/>
+    <parent link="$(arg robot_name)/base_link"/>
+    <child link="$(arg robot_name)/left_wheel"/>
     <axis xyz="0 0 1"/>
   </joint>
   <!-- Right wheel -->
-  <link name="${robot_name}/right_wheel">
+  <link name="$(arg robot_name)/right_wheel">
     <visual>
       <geometry>
@@ -80,12 +80,12 @@
     </inertial>
   </link>
-  <joint name="${robot_name}/right_wheel_joint" type="continuous">
+  <joint name="$(arg robot_name)/right_wheel_joint" type="continuous">
     <origin xyz="0 ${-track_width/2} ${-chassis_height/2 - wheel_width/2}" rpy="0 0 0"/>
-    <parent link="${robot_name}/base_link"/>
-    <child link="${robot_name}/right_wheel"/>
+    <parent link="$(arg robot_name)/base_link"/>
+    <child link="$(arg robot_name)/right_wheel"/>
     <axis xyz="0 0 1"/>
   </joint>
   <!-- Passive caster wheel (sphere) -->
-  <link name="${robot_name}/caster">
+  <link name="$(arg robot_name)/caster">
     <visual>
       <geometry>
@@ -104,19 +104,19 @@
     </inertial>
   </link>
-  <joint name="${robot_name}/caster_joint" type="fixed">
+  <joint name="$(arg robot_name)/caster_joint" type="fixed">
     <origin xyz="${chassis_length/2} 0 ${-chassis_height/2 - caster_radius}" rpy="0 0 0"/>
-    <parent link="${robot_name}/base_link"/>
-    <child link="${robot_name}/caster"/>
+    <parent link="$(arg robot_name)/base_link"/>
+    <child link="$(arg robot_name)/caster"/>
   </joint>
   <!-- Differential drive plugin: accepts /<robot_name>/cmd_vel, publishes /<robot_name>/odom -->
-  <gazebo reference="${robot_name}/base_link">
+  <gazebo reference="$(arg robot_name)/base_link">
     <material>Gazebo/Blue</material>
   </gazebo>
   <gazebo>
     <plugin filename="libgazebo_ros_diff_drive.so" name="gazebo_ros_diff_drive">
-      <robotNamespace>/${robot_name}</robotNamespace>
+      <robotNamespace>/$(arg robot_name)</robotNamespace>
       <updateRate>30</updateRate>
-      <leftJoint>${robot_name}/left_wheel_joint</leftJoint>
-      <rightJoint>${robot_name}/right_wheel_joint</rightJoint>
+      <leftJoint>$(arg robot_name)/left_wheel_joint</leftJoint>
+      <rightJoint>$(arg robot_name)/right_wheel_joint</rightJoint>
       <wheelRadius>${wheel_radius}</wheelRadius>
       <wheelSeparation>${track_width}</wheelSeparation>
@@ -124,5 +124,5 @@
       <odometryTopic>odom</odometryTopic>
       <odometryFrame>odom</odometryFrame>
-      <robotBaseFrame>${robot_name}/base_link</robotBaseFrame>
+      <robotBaseFrame>$(arg robot_name)/base_link</robotBaseFrame>
       <provideOdom>true</provideOdom>
     </plugin>

Commit message: Fix RViz config and simplify box_bot URDF

File: src/nmpc_swarm_demo/urdf/box_bot.urdf.xacro (robot description, xacro)
@@ -1,16 +1,11 @@
 <?xml version="1.0"?>
 <robot xmlns:xacro="http://www.ros.org/wiki/xacro" name="box_bot">
-  <!--
-    Simple lightweight differential-drive robot built from basic geometric
-    primitives. One xacro file is shared by all robots; each spawned instance
-    gets a unique robot_name so its topics sit under /<robot_name>/...
-  -->
   <xacro:arg name="robot_name" default="box_bot"/>
-  <xacro:property name="chassis_length" value="0.30"/>
-  <xacro:property name="chassis_width"  value="0.20"/>
-  <xacro:property name="chassis_height" value="0.10"/>
+  <xacro:property name="chassis_length" value="0.4"/>
+  <xacro:property name="chassis_width"  value="0.3"/>
+  <xacro:property name="chassis_height" value="0.1"/>
   <xacro:property name="wheel_radius"   value="0.06"/>
   <xacro:property name="wheel_width"    value="0.03"/>
-  <xacro:property name="track_width"    value="0.16"/>   <!-- distance between wheels -->
+  <xacro:property name="track_width"    value="0.3"/>
   <xacro:property name="caster_radius"  value="0.03"/>
   <xacro:property name="mass"           value="5.0"/>
@@ -38,5 +33,4 @@
     </inertial>
   </link>
-  <!-- Left wheel -->
   <link name="$(arg robot_name)/left_wheel">
     <visual>
@@ -62,5 +56,4 @@
     <axis xyz="0 0 1"/>
   </joint>
-  <!-- Right wheel -->
   <link name="$(arg robot_name)/right_wheel">
     <visual>
@@ -86,5 +79,4 @@
     <axis xyz="0 0 1"/>
   </joint>
-  <!-- Passive caster wheel (sphere) -->
   <link name="$(arg robot_name)/caster">
     <visual>
@@ -109,5 +101,4 @@
     <child link="$(arg robot_name)/caster"/>
   </joint>
-  <!-- Differential drive plugin: accepts /<robot_name>/cmd_vel, publishes /<robot_name>/odom -->
   <gazebo reference="$(arg robot_name)/base_link">
     <material>Gazebo/Blue</material>

Commit message: Fix RViz NavGoal plugin and URDF root link inertia

File: src/nmpc_swarm_demo/urdf/box_bot.urdf.xacro (robot description, xacro)
@@ -16,4 +16,15 @@
     <color rgba="0.1 0.1 0.1 1.0"/>
   </material>
+  <!-- Dummy root link to avoid KDL root-link inertia warning -->
+  <link name="$(arg robot_name)/dummy_root">
+    <inertial>
+      <mass value="0.001"/>
+      <inertia ixx="0.0001" ixy="0.0" ixz="0.0" iyy="0.0001" iyz="0.0" izz="0.0001"/>
+    </inertial>
+  </link>
+  <joint name="$(arg robot_name)/dummy_root_joint" type="fixed">
+    <parent link="$(arg robot_name)/dummy_root"/>
+    <child link="$(arg robot_name)/base_link"/>
+  </joint>
   <link name="$(arg robot_name)/base_link">
     <visual>

Commit message: Fix robot spawning, TF, RViz display, and NMPC controller
- Fix static_obstacles param parsing (string -> JSON list) - was causing segfault
- Fix path publisher to use PoseStamped instead of Pose
- Add publishTf/publishWheelTF to URDF - enables odom->base_link TF, prevents wheel TF conflicts
- Add dummy base_footprint link - fixes KDL root link inertia warning
- Remove frame_prefix from robot_state_publisher - avoids double-prefixing
- Update RViz RobotModel to use namespaced robot_description params
- Add spawn_robot.sh to clean stale Gazebo entities before respawn
- Set headless=false for user-facing GUI launch

File: src/nmpc_swarm_demo/urdf/box_bot.urdf.xacro (robot description, xacro)
@@ -1,132 +1,315 @@
 <?xml version="1.0"?>
-<robot xmlns:xacro="http://www.ros.org/wiki/xacro" name="box_bot">
-  <xacro:arg name="robot_name" default="box_bot"/>
-  <xacro:property name="chassis_length" value="0.4"/>
-  <xacro:property name="chassis_width"  value="0.3"/>
-  <xacro:property name="chassis_height" value="0.1"/>
-  <xacro:property name="wheel_radius"   value="0.06"/>
-  <xacro:property name="wheel_width"    value="0.03"/>
-  <xacro:property name="track_width"    value="0.3"/>
-  <xacro:property name="caster_radius"  value="0.03"/>
-  <xacro:property name="mass"           value="5.0"/>
-  <material name="blue">
-    <color rgba="0.2 0.4 1.0 1.0"/>
-  </material>
-  <material name="black">
-    <color rgba="0.1 0.1 0.1 1.0"/>
-  </material>
-  <!-- Dummy root link to avoid KDL root-link inertia warning -->
-  <link name="$(arg robot_name)/dummy_root">
-    <inertial>
-      <mass value="0.001"/>
-      <inertia ixx="0.0001" ixy="0.0" ixz="0.0" iyy="0.0001" iyz="0.0" izz="0.0001"/>
-    </inertial>
-  </link>
-  <joint name="$(arg robot_name)/dummy_root_joint" type="fixed">
-    <parent link="$(arg robot_name)/dummy_root"/>
-    <child link="$(arg robot_name)/base_link"/>
-  </joint>
-  <link name="$(arg robot_name)/base_link">
-    <visual>
-      <geometry>
-        <box size="${chassis_length} ${chassis_width} ${chassis_height}"/>
-      </geometry>
-      <material name="blue"/>
-    </visual>
-    <collision>
-      <geometry>
-        <box size="${chassis_length} ${chassis_width} ${chassis_height}"/>
-      </geometry>
-    </collision>
-    <inertial>
-      <mass value="${mass}"/>
-      <inertia ixx="0.05" ixy="0.0" ixz="0.0" iyy="0.05" iyz="0.0" izz="0.08"/>
-    </inertial>
-  </link>
-  <link name="$(arg robot_name)/left_wheel">
-    <visual>
-      <geometry>
-        <cylinder length="${wheel_width}" radius="${wheel_radius}"/>
-      </geometry>
-      <material name="black"/>
-    </visual>
-    <collision>
-      <geometry>
-        <cylinder length="${wheel_width}" radius="${wheel_radius}"/>
-      </geometry>
-    </collision>
-    <inertial>
+<robot name="differential_robot" xmlns:xacro="http://www.ros.org/wiki/xacro">
+  <!-- Prefix argument (e.g., "robot_0/", "robot_1/") -->
+  <xacro:arg name="prefix" default=""/>
+  <!-- Dummy base link (KDL workaround: root link cannot have inertia) -->
+  <link name="$(eval prefix)base_footprint"/>
+  <joint name="$(eval prefix)base_footprint_joint" type="fixed">
+    <parent link="$(eval prefix)base_footprint"/>
+    <child link="$(eval prefix)base_link"/>
+    <origin xyz="0 0 0" rpy="0 0 0"/>
+  </joint>
+  <!-- Link for the main body of the robot -->
+  <link name="$(eval prefix)base_link">
+    <inertial>
+      <origin xyz="0 0 0" rpy="0 0 0"/>
+      <mass value="1.5"/>
+      <inertia ixx="0.02" ixy="0.0" ixz="0.0" iyy="0.04" iyz="0.0" izz="0.07"/>
+    </inertial>
+    <visual>
+      <origin xyz="0 0 0" rpy="0 0 0"/>
+      <geometry>
+        <box size="0.5 0.3 0.1"/>
+      </geometry>
+      <material name="blue">
+        <color rgba="0.0 0.0 0.5 1.0"/>
+      </material>
+    </visual>
+    <collision>
+      <origin xyz="0 0 0" rpy="0 0 0"/>
+      <geometry>
+        <box size="0.5 0.3 0.1"/>
+      </geometry>
+    </collision>
+  </link>
+  <!-- Left wheel -->
+  <link name="$(eval prefix)left_wheel">
+    <inertial>
+      <origin xyz="0 0 0" rpy="1.57 0 0"/>
       <mass value="0.5"/>
-      <inertia ixx="0.001" ixy="0.0" ixz="0.0" iyy="0.001" iyz="0.0" izz="0.001"/>
-    </inertial>
-  </link>
-  <joint name="$(arg robot_name)/left_wheel_joint" type="continuous">
-    <origin xyz="0 ${track_width/2} ${-chassis_height/2 - wheel_width/2}" rpy="0 0 0"/>
-    <parent link="$(arg robot_name)/base_link"/>
-    <child link="$(arg robot_name)/left_wheel"/>
-    <axis xyz="0 0 1"/>
-  </joint>
-  <link name="$(arg robot_name)/right_wheel">
-    <visual>
-      <geometry>
-        <cylinder length="${wheel_width}" radius="${wheel_radius}"/>
-      </geometry>
-      <material name="black"/>
-    </visual>
-    <collision>
-      <geometry>
-        <cylinder length="${wheel_width}" radius="${wheel_radius}"/>
-      </geometry>
-    </collision>
-    <inertial>
+      <inertia ixx="0.0025" ixy="0.0" ixz="0.0" iyy="0.0025" iyz="0.0" izz="0.0025"/>
+    </inertial>
+    <visual>
+      <origin xyz="0 0 0" rpy="1.57 0 0"/>
+      <geometry>
+        <cylinder radius="0.1" length="0.05"/>
+      </geometry>
+      <material name="black">
+        <color rgba="0.0 0.0 0.0 1.0"/>
+      </material>
+    </visual>
+    <collision>
+      <origin xyz="0 0 0" rpy="1.57 0 0"/>
+      <geometry>
+        <cylinder radius="0.1" length="0.05"/>
+      </geometry>
+    </collision>
+  </link>
+  <!-- Right wheel -->
+  <link name="$(eval prefix)right_wheel">
+    <inertial>
+    <origin xyz="0 0 0" rpy="1.57 0 0"/>
       <mass value="0.5"/>
-      <inertia ixx="0.001" ixy="0.0" ixz="0.0" iyy="0.001" iyz="0.0" izz="0.001"/>
-    </inertial>
-  </link>
-  <joint name="$(arg robot_name)/right_wheel_joint" type="continuous">
-    <origin xyz="0 ${-track_width/2} ${-chassis_height/2 - wheel_width/2}" rpy="0 0 0"/>
-    <parent link="$(arg robot_name)/base_link"/>
-    <child link="$(arg robot_name)/right_wheel"/>
-    <axis xyz="0 0 1"/>
-  </joint>
-  <link name="$(arg robot_name)/caster">
-    <visual>
-      <geometry>
-        <sphere radius="${caster_radius}"/>
-      </geometry>
-      <material name="black"/>
-    </visual>
-    <collision>
-      <geometry>
-        <sphere radius="${caster_radius}"/>
-      </geometry>
-    </collision>
-    <inertial>
-      <mass value="0.2"/>
-      <inertia ixx="0.0001" ixy="0.0" ixz="0.0" iyy="0.0001" iyz="0.0" izz="0.0001"/>
-    </inertial>
-  </link>
-  <joint name="$(arg robot_name)/caster_joint" type="fixed">
-    <origin xyz="${chassis_length/2} 0 ${-chassis_height/2 - caster_radius}" rpy="0 0 0"/>
-    <parent link="$(arg robot_name)/base_link"/>
-    <child link="$(arg robot_name)/caster"/>
-  </joint>
-  <gazebo reference="$(arg robot_name)/base_link">
-    <material>Gazebo/Blue</material>
-  </gazebo>
-  <gazebo>
-    <plugin filename="libgazebo_ros_diff_drive.so" name="gazebo_ros_diff_drive">
-      <robotNamespace>/$(arg robot_name)</robotNamespace>
-      <updateRate>30</updateRate>
-      <leftJoint>$(arg robot_name)/left_wheel_joint</leftJoint>
-      <rightJoint>$(arg robot_name)/right_wheel_joint</rightJoint>
-      <wheelRadius>${wheel_radius}</wheelRadius>
-      <wheelSeparation>${track_width}</wheelSeparation>
+      <inertia ixx="0.0025" ixy="0.0" ixz="0.0" iyy="0.0025" iyz="0.0" izz="0.0025"/>
+    </inertial>
+    <visual>
+    <origin xyz="0 0 0" rpy="1.57 0 0"/>
+      <geometry>
+        <cylinder radius="0.1" length="0.05"/>
+      </geometry>
+      <material name="black">
+        <color rgba="0.0 0.0 0.0 1.0"/>
+      </material>
+    </visual>
+    <collision>
+    <origin xyz="0 0 0" rpy="1.57 0 0"/>
+      <geometry>
+        <cylinder radius="0.1" length="0.05"/>
+      </geometry>
+    </collision>
+  </link>
+  <link name="$(eval prefix)caster_wheel">
+    <inertial>
+      <mass value="0.5"/>
+      <inertia ixx="0.0005" ixy="0.0" ixz="0.0" iyy="0.0005" iyz="0.0" izz="0.0005"/>
+    </inertial>
+    <visual>
+      <geometry>
+        <sphere radius="0.05"/>
+      </geometry>
+      <material name="black">
+        <color rgba="0.0 0.0 0.0 1.0"/>
+      </material>
+    </visual>
+    <collision>
+      <geometry>
+        <sphere radius="0.05"/>
+      </geometry>
+    </collision>
+  </link>
+  <!-- Joints for wheels -->
+  <joint name="$(eval prefix)left_wheel_joint" type="continuous">
+    <parent link="$(eval prefix)base_link"/>
+    <child link="$(eval prefix)left_wheel"/>
+    <origin xyz="-0.125 0.175 0" rpy="0 0 0"/>
+    <axis xyz="0 1 0"/>
+  </joint>
+  <joint name="$(eval prefix)right_wheel_joint" type="continuous">
+    <parent link="$(eval prefix)base_link"/>
+    <child link="$(eval prefix)right_wheel"/>
+    <origin xyz="-0.125 -0.175 0" rpy="0 0 0"/>
+    <axis xyz="0 1 0"/>
+  </joint>
+  <joint name="$(eval prefix)caster_wheel_joint" type="fixed">
+    <parent link="$(eval prefix)base_link"/>
+    <child link="$(eval prefix)caster_wheel"/>
+    <origin xyz="0.2 0.0 -0.05" rpy="0 0 0"/>
+  </joint>
+   <gazebo>
+    <plugin name="$(eval prefix)differential_drive_controller" filename="libgazebo_ros_diff_drive.so">
+      <!-- Robot namespace for this robot -->
+      <robotNamespace>$(eval prefix)</robotNamespace>
+      <!-- Plugin update rate in Hz -->
+      <updateRate>10</updateRate>
+      <!-- Name of left joint, defaults to `left_joint` -->
+      <leftJoint>$(eval prefix)left_wheel_joint</leftJoint>
+      <!-- Name of right joint, defaults to `right_joint` -->
+      <rightJoint>$(eval prefix)right_wheel_joint</rightJoint>
+      <!-- The distance from the center of one wheel to the other, in meters, defaults to 0.34 m -->
+      <wheelSeparation>0.2</wheelSeparation>
+      <!-- Diameter of the wheels, in meters, defaults to 0.15 m -->
+      <wheelDiameter>0.2</wheelDiameter>
+      <!-- Wheel acceleration, in rad/s^2, defaults to 0.0 rad/s^2 -->
+      <wheelAcceleration>0.0</wheelAcceleration>
+      <!-- Maximum torque which the wheels can produce, in Nm, defaults to 5 Nm -->
+      <wheelTorque>5</wheelTorque>
+      <!-- Topic to receive geometry_msgs/Twist message commands, defaults to `cmd_vel` -->
       <commandTopic>cmd_vel</commandTopic>
+      <!-- Topic to publish nav_msgs/Odometry messages, defaults to `odom` -->
       <odometryTopic>odom</odometryTopic>
+      <!-- Odometry frame, defaults to `odom` -->
       <odometryFrame>odom</odometryFrame>
-      <robotBaseFrame>$(arg robot_name)/base_link</robotBaseFrame>
-      <provideOdom>true</provideOdom>
+      <!-- Robot frame to calculate odometry from, defaults to `base_footprint` -->
+      <robotBaseFrame>$(eval prefix)base_link</robotBaseFrame>
+      <!-- Odometry source, 0 for ENCODER, 1 for WORLD, defaults to WORLD -->
+      <odometrySource>1</odometrySource>
+      <!-- Set to false to publish transforms for the wheel links, defaults to false -->
+      <publishWheelTF>false</publishWheelTF>
+      <!-- Set to true to publish odom->base_link TF, defaults to true -->
+      <publishTf>true</publishTf>
+      <!-- Set to true to publish sensor_msgs/JointState on /joint_states for the wheel joints, defaults to false -->
+      <publishWheelJointState>true</publishWheelJointState>
+      <!-- Set to true to swap right and left wheels, defaults to true -->
+      <legacyMode>false</legacyMode>
     </plugin>
   </gazebo>
+  <link name="$(eval prefix)camera_link">
+    <visual>
+      <geometry>
+        <box size="0.05 0.05 0.05" />
+      </geometry>
+      <material name="red">
+        <color rgba="0.5 0.0 0.0 1.0" />
+      </material>
+    </visual>
+  </link>
+  <joint name="$(eval prefix)camera_joint" type="fixed">
+    <parent link="$(eval prefix)base_link"/>
+    <child link="$(eval prefix)camera_link"/>
+    <origin xyz="0.275 0.0 0.0" rpy="0 0 0"/>
+  </joint>
+  <gazebo reference="$(eval prefix)camera_link">
+    <material>Gazebo/Red</material>
+    <sensor type="camera" name="camera_sensor">
+      <pose>0 0 0 0 0 0</pose>
+      <camera>
+        <horizontal_fov>1.047</horizontal_fov>
+        <image>
+          <width>640</width>
+          <height>480</height>
+        </image>
+        <clip>
+          <near>0.1</near>
+          <far>100</far>
+        </clip>
+      </camera>
+      <plugin name="$(eval prefix)camera_controller" filename="libgazebo_ros_camera.so">
+        <always_on>true</always_on>
+        <update_rate>6.0</update_rate>
+      </plugin>
+    </sensor>
+  </gazebo>
+  <joint name="$(eval prefix)laser_joint" type="fixed">
+      <parent link="$(eval prefix)base_link"/>
+      <child link="$(eval prefix)laser_link"/>
+      <origin xyz="0.05 0 0.125" rpy="0 0 0"/>
+  </joint>
+  <link name="$(eval prefix)laser_link">
+      <visual>
+          <origin xyz="0 0 -0.05" rpy="0 0 0"/>
+          <geometry>
+              <cylinder radius="0.05" length="0.1"/>
+          </geometry>
+          <material name="red"/>
+      </visual>
+      <collision>
+          <geometry>
+              <cylinder radius="0.05" length="0.1"/>
+          </geometry>
+      </collision>
+      <inertial>
+        <origin xyz="0 0 0" rpy="0 0 0"/>
+        <mass value="0.1"/>
+        <inertia ixx="0.01" ixy="0.0" ixz="0.0" iyy="0.01" iyz="0.0" izz="0.01"/>
+      </inertial>
+  </link>
+  <gazebo reference="$(eval prefix)laser_link">
+    <material>Gazebo/Red</material>
+    <sensor type="ray" name="head_hokuyo_sensor">
+      <pose>0 0 0 0 0 0</pose>
+      <visualize>true</visualize>
+      <update_rate>10</update_rate>
+      <ray>
+        <scan>
+          <horizontal>
+            <samples>360</samples>
+            <resolution>1</resolution>
+            <min_angle>-3.14</min_angle>
+            <max_angle>3.14</max_angle>
+          </horizontal>
+        </scan>
+        <range>
+          <min>0.10</min>
+          <max>6.0</max>
+          <resolution>0.01</resolution>
+        </range>
+        <noise>
+          <type>gaussian</type>
+          <mean>0.0</mean>
+          <stddev>0.01</stddev>
+        </noise>
+      </ray>
+      <plugin name="$(eval prefix)gazebo_ros_head_hokuyo_controller" filename="libgazebo_ros_laser.so">
+        <topicName>$(eval prefix)scan</topicName>
+        <frameName>$(eval prefix)laser_link</frameName>
+      </plugin>
+    </sensor>
+  </gazebo>
+  <gazebo reference="$(eval prefix)base_footprint">
+      <material>Gazebo/Transparent</material>
+  </gazebo>
+  <gazebo reference="$(eval prefix)base_link">
+      <material>Gazebo/Blue</material>
+  </gazebo>
+  <gazebo reference="$(eval prefix)left_wheel">
+      <material>Gazebo/Black</material>
+      <mu1>0.5</mu1>
+      <mu2>0.5</mu2>
+  </gazebo>
+  <gazebo reference="$(eval prefix)right_wheel">
+      <material>Gazebo/Black</material>
+      <mu1>0.5</mu1>
+      <mu2>0.5</mu2>
+  </gazebo>
+  <gazebo reference="$(eval prefix)castor_wheel">
+      <material>Gazebo/Black</material>
+      <mu1>0.001</mu1>
+      <mu2>0.001</mu2>
+  </gazebo>
+  <!-- IMU Sensor -->
+  <link name="$(eval prefix)imu_link">
+    <inertial>
+      <mass value="1.0"/>
+      <inertia ixx="0.00125" ixy="0.0" ixz="0.0" iyy="0.00125" iyz="0.0" izz="0.00125"/>
+    </inertial>
+    <visual>
+      <geometry>
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