Commit message: Fix circling at goal: arrival detection, stronger terminal cost, URDF friction fixes, NMPC cruise control + inverse barriers

File: src/nmpc_swarm_demo/urdf/box_bot.urdf.xacro (robot description, xacro)
@@ -15,5 +15,9 @@
       <origin xyz="0 0 0" rpy="0 0 0"/>
       <mass value="1.5"/>
-      <inertia ixx="0.02" ixy="0.0" ixz="0.0" iyy="0.04" iyz="0.0" izz="0.07"/>
+      <!-- Correct box inertia: 0.5x0.3x0.1, mass=1.5 -->
+      <!-- ixx = 1/12*m*(y^2+z^2) = 0.0125 -->
+      <!-- iyy = 1/12*m*(x^2+z^2) = 0.0325 -->
+      <!-- izz = 1/12*m*(x^2+y^2) = 0.0425 -->
+      <inertia ixx="0.0125" ixy="0.0" ixz="0.0" iyy="0.0325" iyz="0.0" izz="0.0425"/>
     </inertial>
     <visual>
@@ -116,42 +120,42 @@
     <origin xyz="0.2 0.0 -0.05" rpy="0 0 0"/>
   </joint>
-   <gazebo>
-    <plugin name="$(eval prefix)differential_drive_controller" filename="libgazebo_ros_diff_drive.so">
-      <!-- Robot namespace for this robot -->
-      <robotNamespace>$(eval prefix)</robotNamespace>
-      <!-- Plugin update rate in Hz -->
-      <updateRate>10</updateRate>
-      <!-- Name of left joint, defaults to `left_joint` -->
-      <leftJoint>$(eval prefix)left_wheel_joint</leftJoint>
-      <!-- Name of right joint, defaults to `right_joint` -->
-      <rightJoint>$(eval prefix)right_wheel_joint</rightJoint>
-      <!-- The distance from the center of one wheel to the other, in meters, defaults to 0.34 m -->
-      <wheelSeparation>0.2</wheelSeparation>
-      <!-- Diameter of the wheels, in meters, defaults to 0.15 m -->
-      <wheelDiameter>0.2</wheelDiameter>
-      <!-- Wheel acceleration, in rad/s^2, defaults to 0.0 rad/s^2 -->
-      <wheelAcceleration>0.0</wheelAcceleration>
-      <!-- Maximum torque which the wheels can produce, in Nm, defaults to 5 Nm -->
-      <wheelTorque>5</wheelTorque>
-      <!-- Topic to receive geometry_msgs/Twist message commands, defaults to `cmd_vel` -->
-      <commandTopic>cmd_vel</commandTopic>
-      <!-- Topic to publish nav_msgs/Odometry messages, defaults to `odom` -->
-      <odometryTopic>odom</odometryTopic>
-      <!-- Odometry frame, defaults to `odom` -->
-      <odometryFrame>odom</odometryFrame>
-      <!-- Robot frame to calculate odometry from, defaults to `base_footprint` -->
-      <robotBaseFrame>$(eval prefix)base_link</robotBaseFrame>
-      <!-- Odometry source, 0 for ENCODER, 1 for WORLD, defaults to WORLD -->
-      <odometrySource>1</odometrySource>
-      <!-- Set to false to publish transforms for the wheel links, defaults to false -->
-      <publishWheelTF>false</publishWheelTF>
-      <!-- Set to true to publish odom->base_link TF, defaults to true -->
-      <publishTf>true</publishTf>
-      <!-- Set to true to publish sensor_msgs/JointState on /joint_states for the wheel joints, defaults to false -->
-      <publishWheelJointState>true</publishWheelJointState>
-      <!-- Set to true to swap right and left wheels, defaults to true -->
-      <legacyMode>false</legacyMode>
-    </plugin>
-  </gazebo>
+<gazebo>
+     <plugin name="$(eval prefix)differential_drive_controller" filename="libgazebo_ros_diff_drive.so">
+       <!-- Robot namespace for this robot -->
+       <robotNamespace>$(eval prefix)</robotNamespace>
+       <!-- Plugin update rate in Hz -->
+       <updateRate>100</updateRate>
+       <!-- Name of left joint, defaults to `left_joint` -->
+       <leftJoint>$(eval prefix)left_wheel_joint</leftJoint>
+       <!-- Name of right joint, defaults to `right_joint` -->
+       <rightJoint>$(eval prefix)right_wheel_joint</rightJoint>
+       <!-- The distance from the center of one wheel to the other, in meters, defaults to 0.34 m -->
+       <wheelSeparation>0.35</wheelSeparation>
+       <!-- Diameter of the wheels, in meters, defaults to 0.15 m -->
+       <wheelDiameter>0.2</wheelDiameter>
+       <!-- Wheel acceleration, in rad/s^2, defaults to 0.0 rad/s^2 -->
+       <wheelAcceleration>10.0</wheelAcceleration>
+       <!-- Maximum torque which the wheels can produce, in Nm, defaults to 5 Nm -->
+       <wheelTorque>20</wheelTorque>
+       <!-- Topic to receive geometry_msgs/Twist message commands, defaults to `cmd_vel` -->
+       <commandTopic>cmd_vel</commandTopic>
+       <!-- Topic to publish nav_msgs/Odometry messages, defaults to `odom` -->
+       <odometryTopic>odom</odometryTopic>
+       <!-- Odometry frame, defaults to `odom` -->
+       <odometryFrame>odom</odometryFrame>
+       <!-- Robot frame to calculate odometry from, defaults to `base_footprint` -->
+       <robotBaseFrame>$(eval prefix)base_link</robotBaseFrame>
+       <!-- Odometry source, 0 for ENCODER, 1 for WORLD, defaults to WORLD -->
+       <odometrySource>1</odometrySource>
+       <!-- Set to false to publish transforms for the wheel links, defaults to false -->
+       <publishWheelTF>false</publishWheelTF>
+       <!-- Set to true to publish odom->base_link TF, defaults to true -->
+       <publishTf>true</publishTf>
+       <!-- Set to true to publish sensor_msgs/JointState on /joint_states for the wheel joints, defaults to false -->
+       <publishWheelJointState>true</publishWheelJointState>
+       <!-- Set to true to swap right and left wheels, defaults to true -->
+       <legacyMode>false</legacyMode>
+     </plugin>
+   </gazebo>
   <link name="$(eval prefix)camera_link">
     <visual>
@@ -252,19 +256,27 @@
       <material>Gazebo/Blue</material>
   </gazebo>
-  <gazebo reference="$(eval prefix)left_wheel">
+<gazebo reference="$(eval prefix)left_wheel">
       <material>Gazebo/Black</material>
-      <mu1>0.5</mu1>
-      <mu2>0.5</mu2>
-  </gazebo>
-  <gazebo reference="$(eval prefix)right_wheel">
+      <mu1>1.0</mu1>
+      <mu2>1.0</mu2>
+      <fdir1>1 0 0</fdir1>
+      <kp>1000000.0</kp>
+      <kd>100.0</kd>
+    </gazebo>
+    <gazebo reference="$(eval prefix)right_wheel">
       <material>Gazebo/Black</material>
-      <mu1>0.5</mu1>
-      <mu2>0.5</mu2>
-  </gazebo>
-  <gazebo reference="$(eval prefix)castor_wheel">
+      <mu1>1.0</mu1>
+      <mu2>1.0</mu2>
+      <fdir1>1 0 0</fdir1>
+      <kp>1000000.0</kp>
+      <kd>100.0</kd>
+    </gazebo>
+    <gazebo reference="$(eval prefix)caster_wheel">
       <material>Gazebo/Black</material>
-      <mu1>0.001</mu1>
-      <mu2>0.001</mu2>
-  </gazebo>
+      <mu1>0.0</mu1>
+      <mu2>0.0</mu2>
+      <slip1>1.0</slip1>
+      <slip2>1.0</slip2>
+    </gazebo>
   <!-- IMU Sensor -->
   <link name="$(eval prefix)imu_link">
